File: IOB-Adapter-Minimal_array.brd (EAGLE design)
At the start: 99.1 x 96.5 mm, 60 parts

Commit message: normalized values
Parts:
- JP1X11, JP1X110, JP1X12, JP1X13, JP1X14, JP1X15, JP1X16, JP1X17, JP1X18, JP1X19, JP1X21, JP1X210, JP1X22, JP1X23, JP1X24, JP1X25, JP1X26, JP1X27, JP1X28, JP1X29, JP1X31, JP1X310, JP1X32, JP1X33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: value CONNECTOR-M05X2NO_SILK -> 0.100
